File: hardware/USB.kicad_sch (KiCad schematic)
At the start: 0 parts

Commit message: poop
Other:
- note added: "Will probably use: CP2102N-A02-GQFN20 for USB-UART TUSB1210 for OTG Something like CH224K for USB-PD?"
Changed lines of the file:
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@@
+		)
+	)
+	(text "Will probably use:\n	CP2102N-A02-GQFN20 for USB-UART\n	TUSB1210 for OTG\n	Something like CH224K for USB-PD?"
+		(exclude_from_sim no)
+		(at 40.132 64.77 0)
+		(effects
+			(font
+				(size 3 3)
+				(thickness 0.6)
+				(bold yes)
+			)
+			(justify left)
 		)
 	)
