File: hardware/ZED.kicad_sch (KiCad schematic)
At the start: 1 part, among them U2 XC7Z020-1CLG484C

Commit message: starting layout
Parts:
- removed U2: XC7Z020-1CLG484C, CLG484_XIL, symbol XC7Z020_1CLG484C:XC7Z020-1CLG484C
