File: hardware/pmod.kicad_sch (KiCad schematic)
At the start: 4 parts, among them J1 Conn_02x06_Top_Bottom, J2 Conn_02x06_Top_Bottom, J3 Conn_02x06_Top_Bottom, J4 Conn_02x06_Top_Bottom

Commit message: matthew review or get touched
Changed lines of the file:
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@@
 	(wire
 		(pts
-			(xy 132.08 39.37) (xy 134.62 39.37)
-		)
-		(stroke
-			(width 0)
-			(type default)
-		)
-	)
-	(wire
-		(pts
-			(xy 132.08 69.85) (xy 134.62 69.85)
-		)
-		(stroke
-			(width 0)
-			(type default)
-		)
-	)
-	(wire
-		(pts
 			(xy 195.58 74.93) (xy 198.12 74.93)
 		)
@@
 	(wire
 		(pts
-			(xy 182.88 34.29) (xy 168.91 34.29)
+			(xy 132.08 39.37) (xy 137.16 39.37)
 		)
 		(stroke
@@
 	(wire
 		(pts
-			(xy 209.55 34.29) (xy 209.55 36.83)
+			(xy 182.88 34.29) (xy 168.91 34.29)
 		)
 		(stroke
@@
 	(wire
 		(pts
-			(xy 105.41 34.29) (xy 105.41 36.83)
+			(xy 209.55 34.29) (xy 209.55 36.83)
 		)
 		(stroke
@@
 	(wire
 		(pts
-			(xy 168.91 64.77) (xy 168.91 67.31)
+			(xy 105.41 34.29) (xy 105.41 36.83)
 		)
 		(stroke
@@
 	(wire
 		(pts
-			(xy 140.97 59.69) (xy 140.97 62.23)
+			(xy 168.91 64.77) (xy 168.91 67.31)
 		)
 		(stroke
@@
 	(wire
 		(pts
-			(xy 195.58 62.23) (xy 204.47 62.23)
+			(xy 140.97 59.69) (xy 140.97 62.23)
 		)
 		(stroke
@@
 	(wire
 		(pts
-			(xy 132.08 44.45) (xy 134.62 44.45)
+			(xy 195.58 62.23) (xy 204.47 62.23)
 		)
 		(stroke
@@
 	(wire
 		(pts
-			(xy 179.07 72.39) (xy 182.88 72.39)
+			(xy 132.08 41.91) (xy 137.16 41.91)
 		)
 		(stroke
@@
 	(wire
 		(pts
-			(xy 179.07 67.31) (xy 182.88 67.31)
+			(xy 179.07 72.39) (xy 182.88 72.39)
 		)
 		(stroke
@@
 	(wire
 		(pts
-			(xy 115.57 67.31) (xy 119.38 67.31)
+			(xy 179.07 67.31) (xy 182.88 67.31)
 		)
 		(stroke
@@
 	(wire
 		(pts
-			(xy 119.38 64.77) (xy 105.41 64.77)
+			(xy 114.3 67.31) (xy 119.38 67.31)
 		)
 		(stroke
@@
 	(wire
 		(pts
-			(xy 195.58 64.77) (xy 209.55 64.77)
+			(xy 119.38 64.77) (xy 105.41 64.77)
 		)
 		(stroke
@@
 	(wire
 		(pts
-			(xy 132.08 67.31) (xy 134.62 67.31)
+			(xy 195.58 64.77) (xy 209.55 64.77)
 		)
 		(stroke
@@
 	(wire
 		(pts
-			(xy 132.08 36.83) (xy 134.62 36.83)
+			(xy 132.08 36.83) (xy 137.16 36.83)
 		)
 		(stroke
@@
 	(wire
 		(pts
-			(xy 132.08 74.93) (xy 134.62 74.93)
-		)
-		(stroke
-			(width 0)
-			(type default)
-		)
-	)
-	(wire
-		(pts
-			(xy 132.08 41.91) (xy 134.62 41.91)
+			(xy 182.88 31.75) (xy 173.99 31.75)
 		)
 		(stroke
@@
 	(wire
 		(pts
-			(xy 182.88 31.75) (xy 173.99 31.75)
+			(xy 114.3 74.93) (xy 119.38 74.93)
 		)
 		(stroke
@@
 	(wire
 		(pts
-			(xy 115.57 74.93) (xy 119.38 74.93)
+			(xy 179.07 74.93) (xy 182.88 74.93)
 		)
 		(stroke
@@
 	(wire
 		(pts
-			(xy 179.07 74.93) (xy 182.88 74.93)
+			(xy 195.58 69.85) (xy 198.12 69.85)
 		)
 		(stroke
@@
 	(wire
 		(pts
-			(xy 195.58 69.85) (xy 198.12 69.85)
+			(xy 195.58 39.37) (xy 198.12 39.37)
 		)
 		(stroke
@@
 	(wire
 		(pts
-			(xy 195.58 39.37) (xy 198.12 39.37)
+			(xy 195.58 41.91) (xy 198.12 41.91)
 		)
 		(stroke
@@
 	(wire
 		(pts
-			(xy 195.58 41.91) (xy 198.12 41.91)
+			(xy 132.08 34.29) (xy 146.05 34.29)
 		)
 		(stroke
@@
 	(wire
 		(pts
-			(xy 132.08 34.29) (xy 146.05 34.29)
+			(xy 132.08 44.45) (xy 137.16 44.45)
 		)
 		(stroke
@@
 	(wire
 		(pts
-			(xy 204.47 29.21) (xy 204.47 31.75)
+			(xy 132.08 67.31) (xy 135.89 67.31)
 		)
 		(stroke
@@
 	(wire
 		(pts
-			(xy 132.08 72.39) (xy 134.62 72.39)
+			(xy 204.47 29.21) (xy 204.47 31.75)
 		)
 		(stroke
@@
 	(wire
 		(pts
-			(xy 115.57 72.39) (xy 119.38 72.39)
+			(xy 114.3 72.39) (xy 119.38 72.39)
+		)
+		(stroke
+			(width 0)
+			(type default)
+		)
+	)
+	(wire
+		(pts
+			(xy 132.08 74.93) (xy 135.89 74.93)
+		)
+		(stroke
+			(width 0)
+			(type default)
+		)
+	)
+	(wire
+		(pts
+			(xy 132.08 69.85) (xy 135.89 69.85)
 		)
 		(stroke
@@
 	(wire
 		(pts
-			(xy 115.57 69.85) (xy 119.38 69.85)
+			(xy 114.3 69.85) (xy 119.38 69.85)
 		)
 		(stroke
@@
 	(wire
 		(pts
+			(xy 132.08 72.39) (xy 135.89 72.39)
+		)
+		(stroke
+			(width 0)
+			(type default)
+		)
+	)
+	(wire
+		(pts
 			(xy 179.07 36.83) (xy 182.88 36.83)
 		)
@@
 	(hierarchical_label "JB10"
 		(shape output)
-		(at 115.57 67.31 180)
+		(at 114.3 67.31 180)
 		(effects
 			(font
@@
 	(hierarchical_label "JB1"
 		(shape output)
-		(at 134.62 74.93 0)
+		(at 135.89 74.93 0)
 		(effects
 			(font
@@
 	(hierarchical_label "JB3"
 		(shape output)
-		(at 134.62 69.85 0)
+		(at 135.89 69.85 0)
 		(effects
 			(font
@@
 	(hierarchical_label "JB9"
 		(shape output)
-		(at 115.57 69.85 180)
+		(at 114.3 69.85 180)
 		(effects
 			(font
@@
 	(hierarchical_label "JA4"
 		(shape output)
-		(at 134.62 36.83 0)
+		(at 137.16 36.83 0)
 		(effects
 			(font
@@
 	(hierarchical_label "JB4"
 		(shape output)
-		(at 134.62 67.31 0)
+		(at 135.89 67.31 0)
 		(effects
 			(font
@@
 	(hierarchical_label "JA3"
 		(shape output)
-		(at 134.62 39.37 0)
+		(at 137.16 39.37 0)
 		(effects
 			(font
@@
 	(hierarchical_label "JB8"
 		(shape output)
-		(at 115.57 72.39 180)
+		(at 114.3 72.39 180)
 		(effects
 			(font
@@
 	(hierarchical_label "JA2"
 		(shape output)
-		(at 134.62 41.91 0)
+		(at 137.16 41.91 0)
 		(effects
 			(font
@@
 	(hierarchical_label "JB2"
 		(shape output)
-		(at 134.62 72.39 0)
+		(at 135.89 72.39 0)
 		(effects
 			(font
@@
 	(hierarchical_label "JB7"
 		(shape output)
-		(at 115.57 74.93 180)
+		(at 114.3 74.93 180)
 		(effects
 			(font
@@
 	(hierarchical_label "JA1"
 		(shape output)
-		(at 134.62 44.45 0)
+		(at 137.16 44.45 0)
 		(effects
 			(font

Commit message: starting layout
Parts:
- J1, J2, J3, J4: footprint (none) -> Connector_PinHeader_2.54mm:PinHeader_2x06_P2.54mm_Horizontal
Changed lines of the file:
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@@
 			)
 		)
-		(property "Footprint" ""
+		(property "Footprint" "Connector_PinHeader_2.54mm:PinHeader_2x06_P2.54mm_Horizontal"
 			(at 190.5 39.37 0)
 			(hide yes)
@@
 			)
 		)
-		(property "Footprint" ""
+		(property "Footprint" "Connector_PinHeader_2.54mm:PinHeader_2x06_P2.54mm_Horizontal"
 			(at 127 39.37 0)
 			(hide yes)
@@
 			)
 		)
-		(property "Footprint" ""
+		(property "Footprint" "Connector_PinHeader_2.54mm:PinHeader_2x06_P2.54mm_Horizontal"
 			(at 127 69.85 0)
 			(hide yes)
@@
 			)
 		)
-		(property "Footprint" ""
+		(property "Footprint" "Connector_PinHeader_2.54mm:PinHeader_2x06_P2.54mm_Horizontal"
 			(at 190.5 69.85 0)
 			(hide yes)
