File: hardware/Ethernet.kicad_sch (KiCad schematic)
At the start: 3 parts, among them IC1 DP83826AIRHBR, J1 RJ45, U2 XC7Z020-1CLG484C

Commit message: poop
Parts:
- removed U2: XC7Z020-1CLG484C, CLG484_XIL, symbol XC7Z020_1CLG484C:XC7Z020-1CLG484C
Other:
- note added: "1. PWR VDDA3V3 = 3.3 V VDDIO = 1.8 V or 3.3 V. (1.8V is strongly considered) 2. CLK A - PHY is RMII leader 25MHz OSC to DP. Chip Generates 50MHz RMII CLK B - RMII follower Gen 50MHz CLK from FPGA and feed 3. Magnetics - ??? Look into this, there seems to be some fuckery An option would be using a MagJack (RJ45 w/ Magnetics) Pulse HX1198FNL or something as well? --- Extra --- 4. RBIAS - 6.49kOhm 5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"
- note added: "Just a heads up: Ss far I have shown 2 options, DP83826I & DP83822I Seems that x26 has been chosen, why? (Curious) Biggest diff that I found is RGMII support This is important because current ZED implements thru RGMII We would be deviating from that using RMII. This is OK, just making sure it is known, and there is plan on how this will be implemented"
- moved on the sheet: IC1

Commit message: finished ethernet
Parts:
- removed J1: RJ45, symbol Connector:RJ45
- added C1, C5: 10u, symbol Device:C
- added C10, C3, C7: 0.1u, symbol Device:C
- added C11, C12, C9: 2n, symbol Device:C
- added C2, C6: 1u, symbol Device:C
- added C4, C8: 0.01u, symbol Device:C
- added D1, D2: LED, symbol Device:LED
- added FB1, FB2: FerriteBead, symbol Device:FerriteBead
- added J5: RJ45_Pulse_JXD6-0001NL, Connector_RJ:RJ45_Pulse_JXD6-0001NL_Horizontal, symbol Connector:RJ45_Pulse_JXD6-0001NL
- added R1: 6.49k, symbol Device:R
- added R2, R3: 1k, symbol Device:R
- added R4, R5: 2.49k, symbol Device:R
- added R6, R7: 4.7k, symbol Device:R
- added R8: 10k, symbol Device:R
- added Y1: SiT8008AI-32-33E-50.000000, SiT8921BM3233N127872000, symbol SiT8008AI-32-33E-50_000000:SiT8008AI-32-33E-50.000000
Connections:
- net GND: now reaches IC1.1 (MODESELECT)
- net GND: now also IC1.33 (EP), C1.2, C10.2, C11.2, C12.2, C2.2, C3.2, C4.2, C5.2, C6.2, C7.2, C8.2, C9.2, R1.2, Y1.2 (GND)
- net at IC1.10 (RBIAS): now also R1.1
- net MDIO: now reaches IC1.11 (MDIO)
- net MDIO: now also R6.2
- net MDC: now reaches IC1.12 (MDC)
- net ETH_RXD1: now reaches IC1.15 (STRAP9/RX_D1)
- net ETH_RXDO: now reaches IC1.16 (STRAP0/RX_D0)
- net VDDIO: now reaches IC1.17 (VDDIO)
- net VDDIO: now also C5.1, C6.1, C7.1, C8.1, FB2.2, R4.1, R5.1, R6.1, R7.1, R8.1
- net ETH_CRS_DV: now reaches IC1.18 (RX_DV/CRS_DV/STRAP10)
- net ETH_CRS_DV: now also R4.2
- net at IC1.2 (CEXT): now also C9.1
- net PHY_INT: now reaches IC1.21 (PWRDN/INT)
- net PHY_INT: now also R7.2
- net ETH_TX_EN: now reaches IC1.23 (TX_EN)
- net ETH_TXD0: now reaches IC1.24 (TX_D0)
- net ETH_TXD1: now reaches IC1.25 (TX_D1)
- net at IC1.28 (COL/LED2/TX_ER/GPIO/STRAP4): now also R5.2
- net VDDA3v3: now reaches IC1.3 (VDDA3V3)
- net VDDA3v3: now also C1.1, C2.1, C3.1, C4.1, FB1.2
- net LED0: now reaches IC1.30 (LED0/STRAP2)
- net LED0: now also R2.2
- net LED1: now reaches IC1.31 (CLKOUT/LED1/STRAP1)
- net LED1: now also R3.2
- net PHY_RST_N: now reaches IC1.32 (RST_N)
- net PHY_RST_N: now also R8.2
- net RD-: now reaches IC1.4 (RD_M)
- net RD-: now also J5.7 (RD-)
- net RD+: now reaches IC1.5 (RD_P)
- net RD+: now also J5.6 (RD+)
- net TD-: now reaches IC1.6 (TD_M)
- net TD-: now also J5.5 (TD-)
- net TD+: now reaches IC1.7 (TD_P)
- net TD+: now also J5.4 (TD+)
- net RMII_REF_CLK: now reaches IC1.9 (XI/50MHZIN)
- net RMII_REF_CLK: now also Y1.3 (OUT)
- new net: D2.1 (K), R3.1
- new net: D1.1 (K), R2.1
- new net: C12.1, J5.8 (RCT)
- new net: C11.1, J5.3 (TCT)
- new net +3.3V: C10.1, D1.2 (A), D2.2 (A), FB1.1, FB2.1, Y1.1 (OE/~{ST}/NC), Y1.4 (VDD)
- new net shield: J5.SH
- no-connect marks 0 -> 1
Other:
- note added: "1% precision resistor required"
- note added: "Going with x26 because we don't need RGMII because too complicated and we don't need 1 gb speeds. Plan is running MPEG/MJPEG which is ~15 mbps so chill"
- note added: "Karthik Notes:"
- note added: "LED 0 indicates activity + Link LED 1 is on when link is 100 mbps Off when link isnt connected or at 10 mbps"
- note added: "Mika Notes:"
- note added: "Power"
- moved on the sheet: IC1

Commit message: some changes`
Parts:
- removed D1, D2: LED, symbol Device:LED
- removed R3: 1k, symbol Device:R
- added C19: 4.7n, symbol Device:C
- added R12, R13: 1k, symbol Device:R
- R2: value 1k -> 1M
Connections:
- net +3.3V: now also J5.10, J5.2
- net GND: now also R2.2, C19.2
- net LED0: now also R13.2; no longer R2.2
- net LED1: now also R12.2
- net shield: now also R2.1, C19.1
- net at J5.1: now also R13.1
- net at J5.9: now also R12.1
- no-connect marks 1 -> 6
Other:
- note added: "FPGA PHY TXD [1:0] -------> Transmit Data TX_EN -------> Transmit valid / enable RXD[1:0] -------> Recieve Data CRS_DV <------- recieve valid REF CLK <------> Clock MDIO/MDC <------> optional configuration/status"

Commit message: clock added
Parts:
- C19, R2: now not fitted
Connections:
- no-connect marks 6 -> 9
Changed lines of the file:
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@@
 	)
 	(no_connect
+		(at 114.3 39.37)
+	)
+	(no_connect
 		(at 139.7 92.71)
 	)
@@
 	)
 	(no_connect
+		(at 106.68 39.37)
+	)
+	(no_connect
 		(at 106.68 125.73)
 	)
 	(no_connect
+		(at 111.76 39.37)
+	)
+	(no_connect
 		(at 73.66 100.33)
 	)
@@
 		(on_board yes)
 		(in_pos_files yes)
-		(dnp no)
+		(dnp yes)
 		(fields_autoplaced yes)
 		(property "Reference" "R2"
@@
 			)
 		)
-		(property "Datasheet" "https://productfinder.pulseeng.com/doc_type/WEB301/doc_num/JXD6-0001NL/doc_part/JXD6-0001NL.pdf"
+		(property "Datasheet" "https://www.mouser.com/datasheet/3/203/1/JXD6_0001NL.pdf"
 			(at 250.19 68.58 0)
 			(hide yes)
@@
 		(on_board yes)
 		(in_pos_files yes)
-		(dnp no)
+		(dnp yes)
 		(fields_autoplaced yes)
 		(property "Reference" "C19"

Commit message: matthew review or get touched
Parts:
- C19, R2: now fitted
Changed lines of the file:
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@@
 		(on_board yes)
 		(in_pos_files yes)
-		(dnp yes)
+		(dnp no)
 		(fields_autoplaced yes)
 		(property "Reference" "R2"
@@
 		(on_board yes)
 		(in_pos_files yes)
-		(dnp yes)
+		(dnp no)
 		(fields_autoplaced yes)
 		(property "Reference" "C19"

Commit message: starting layout
Parts:
- added J8: Conn_01x04, Connector_PinHeader_2.54mm:PinHeader_1x04_P2.54mm_Vertical, symbol Connector_Generic:Conn_01x04
- C1, C10, C11, C12, C19, C2, C3, C4, C5, C6, C7, C8, C9: footprint (none) -> Capacitor_SMD:C_0603_1608Metric_Pad1.08x0.95mm_HandSolder
- FB1, FB2: footprint (none) -> Capacitor_SMD:C_0603_1608Metric_Pad1.08x0.95mm_HandSolder; P/N (none) -> MPZ2012S601ATD25
- IC1: footprint QFN50P500X500X100-33N-D -> DP83826AERHBR:QFN50P500X500X100-33N-D
- R1, R12, R13, R2, R4, R5, R6, R7, R8: footprint (none) -> Resistor_SMD:R_0603_1608Metric_Pad0.98x0.95mm_HandSolder
- Y1: footprint SiT8921BM3233N127872000 -> SiTime SiT8008AI-32-33E-50.000000:SiT8921BM3233N127872000
Connections:
- net RX_ERROR: now reaches IC1.20 (RX_ER/STRAP6)
- net RX_ERROR: now also J8.1 (Pin_1)
- no-connect marks 9 -> 11
Other:
- moved on the sheet: R4

Commit message: most of layout is done, only have single ended highspeed signals left. mika pleaaaaaaaaaaaaaaaaaseeeeeeee review :beg:
Other:
- note removed: "FPGA PHY TXD [1:0] -------> Transmit Data TX_EN -------> Transmit valid / enable RXD[1:0] -------> Recieve Data CRS_DV <------- recieve valid REF CLK <------> Clock MDIO/MDC <------> optional configuration/status"
Changed lines of the file:
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@@
-		)
-	)
-	(text "FPGA			PHY\nTXD [1:0] -------> Transmit Data\nTX_EN     -------> Transmit valid / enable\nRXD[1:0]  -------> Recieve Data\nCRS_DV    <------- recieve valid\nREF CLK   <------> Clock\nMDIO/MDC  <------> optional configuration/status"
-		(exclude_from_sim no)
-		(at 143.764 122.174 0)
-		(effects
-			(font
-				(size 2 2)
-				(thickness 0.4)
-				(bold yes)
-			)
-			(justify left)
 		)
 	)
