File: hardware/OTTER.kicad_pcb (KiCad board)
At the start: 2 copper layers, 51 parts, among them J1 Conn_02x06_Top_Bottom, J2 Conn_02x06_Top_Bottom, J5 RJ45_Pulse_JXD6-0001NL, J6 Conn_01x04, J7 USB_C_Receptacle_USB2.0_14P, U1 TCAN4551RGYRQ1, U4 CH221K

Commit message: some sort of placement done, need to fix up a lott...
Parts:
- added IC1: DP83826AIRHBR, DP83826AERHBR:QFN50P500X500X100-33N-D, F.Cu at (178.8, 35.0)
- added J8: Conn_01x04, Connector_PinHeader_2.54mm:PinHeader_1x04_P2.54mm_Vertical, F.Cu at (172.8, 26.8)
- added R18: 22, Resistor_SMD:R_0603_1608Metric_Pad0.98x0.95mm_HandSolder, F.Cu at (237.1, 44.0)
- added R19: 22, Resistor_SMD:R_0603_1608Metric_Pad0.98x0.95mm_HandSolder, F.Cu at (237.0, 45.5)
- added R20: 22, Resistor_SMD:R_0603_1608Metric_Pad0.98x0.95mm_HandSolder, F.Cu at (237.0, 47.0)
- added R21: 22, Resistor_SMD:R_0603_1608Metric_Pad0.98x0.95mm_HandSolder, F.Cu at (237.0, 48.5)
- added U2: USBLC6-4SC6, Package_TO_SOT_SMD:SOT-23-6, F.Cu at (253.4, 49.0)
- added Y1: SiT8008AI-32-33E-50.000000, SiTime SiT8008AI-32-33E-50.000000:SiT8921BM3233N127872000, F.Cu at (179.2, 27.9)
- added Y3: 7M40000005, 7M40000005:7M27120MAAJT, F.Cu at (239.3, 38.9)
- C20, C21: value 12p -> 10p
- J1, J2: footprint Connector_PinSocket_2.54mm:PinSocket_2x06_P2.54mm_Horizontal -> Connector_PinHeader_2.54mm:PinHeader_2x06_P2.54mm_Horizontal
- R9: value 4.7k -> 10k
- moved J1 150.4 mm to (262.5, 38.0), turned to 0 degrees
- moved C18 131.3 mm to (245.5, 45.5)
- moved C17 129.7 mm to (245.5, 47.0)
- moved R10 129.3 mm to (248.2, 44.0), turned to 180 degrees
- moved J2 128.9 mm to (262.5, 60.9), turned to 0 degrees
- moved C14 128.7 mm to (245.7, 42.6), turned to 90 degrees
- moved C16 128.2 mm to (245.9, 49.5), turned to -90 degrees
- moved C13 126.4 mm to (244.2, 42.6), turned to 90 degrees
- moved C15 126.0 mm to (244.4, 49.5), turned to -90 degrees
- moved C21 121.0 mm to (241.7, 42.5)
- moved U1 119.4 mm to (241.2, 46.1)
- moved C20 116.8 mm to (238.2, 42.5), turned to 180 degrees
- moved R3 115.8 mm to (239.0, 52.4)
- moved R9 113.8 mm to (234.9, 50.0)
- moved JP1 107.4 mm to (241.5, 55.4), turned to -90 degrees
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Connections:
- C15 pad 1: +20v -> +20V
- C16 pad 1: +20v -> +20V
- J1 pad 1: /PMOD Connector/JC1 -> /Ethernet/MDIO
- J1 pad 10: /Ethernet/MDC -> /PMOD Connector/JC10
- J1 pad 2: /PMOD Connector/JC2 -> /Ethernet/MDC
- J1 pad 3: /PMOD Connector/JC3 -> /Ethernet/PHY_INT
- J1 pad 7: /Ethernet/PHY_INT -> /PMOD Connector/JC7
- J1 pad 8: /Ethernet/PHY_RST_N -> /PMOD Connector/JC8
- J1 pad 9: /Ethernet/MDIO -> /PMOD Connector/JC9
- J2 pad 1: /PMOD Connector/JD1 -> /Ethernet/PHY_RST_N
- J2 pad 10: /Ethernet/ETH_TXD0 -> /Ethernet/ETH_TXD1
- J2 pad 2: /Ethernet/ETH_CRS_DV -> /Ethernet/ETH_RXDO
- J2 pad 3: /Ethernet/ETH_RXD1 -> /Ethernet/ETH_TX_EN
- J2 pad 4: /Ethernet/ETH_RXDO -> /Ethernet/ETH_TXD0
- J2 pad 8: /Ethernet/ETH_TX_EN -> /Ethernet/ETH_RXD1
- J2 pad 9: /Ethernet/ETH_TXD1 -> /Ethernet/ETH_CRS_DV
- J6 pad 4: +12V -> +20V
- R10 pad 1: /PMOD Connector/JC2 -> /PMOD Connector/JC8
- R16 pad 1: Net-(U4-VDD) -> /Periphs/USBPD/VDD
- R17 pad 1: Net-(U4-VDD) -> /Periphs/USBPD/VDD
- R9 pad 2: /PMOD Connector/JD1 -> /PMOD Connector/JC10
- U1 pad 14: +20v -> +20V
- U1 pad 19: /PMOD Connector/JC2 -> /PMOD Connector/JC8
- U1 pad 4: /PMOD Connector/JC3 -> Net-(U1-SCLK)
- U1 pad 5: /PMOD Connector/JC4 -> Net-(U1-SDI)
- U1 pad 6: /PMOD Connector/JC1 -> Net-(U1-SDO)
- U1 pad 7: /PMOD Connector/JD1 -> Net-(U1-~{CS})
- U4 pad 1: Net-(U4-VDD) -> /Periphs/USBPD/VDD
Other:
- copper layers 2 -> 4

Commit message: inital layout review
Parts:
- removed J6: Conn_01x04, Connector_PinSocket_2.54mm:PinSocket_1x04_P2.54mm_Vertical
- removed J8: Conn_01x04, Connector_PinHeader_2.54mm:PinHeader_1x04_P2.54mm_Vertical
- removed JP1: Jumper_2_Small_Open, Connector_PinHeader_2.54mm:PinHeader_1x02_P2.54mm_Vertical
- removed R3: 120, Resistor_SMD:R_0603_1608Metric_Pad0.98x0.95mm_HandSolder
- moved C5 68.4 mm to (220.2, 57.3), turned to 90 degrees
- moved C7 65.7 mm to (217.8, 56.4)
- moved C6 65.5 mm to (217.8, 58.2), turned to 180 degrees
- moved FB2 63.6 mm to (220.5, 59.9), turned to 180 degrees
- moved C8 62.7 mm to (215.2, 57.3), turned to -90 degrees
- moved C4 55.2 mm to (207.2, 51.9), turned to 90 degrees
- moved R4 54.9 mm to (216.6, 53.9), turned to -90 degrees
- moved C2 54.5 mm to (204.8, 51.1)
- moved C3 54.1 mm to (204.8, 52.6), turned to 180 degrees
- moved C10 53.9 mm to (204.5, 63.1)
- moved C1 53.7 mm to (202.2, 51.9), turned to -90 degrees
- moved J7 52.6 mm to (230.8, 46.6), turned to 180 degrees
- moved R6 52.4 mm to (210.5, 59.4), turned to 90 degrees
- moved R1 51.8 mm to (208.8, 59.4), turned to -90 degrees
- moved R7 51.7 mm to (215.1, 52.9), turned to -90 degrees
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Routing:
- net /Ethernet/MDIO: track 0.00 -> 1.62 mm
- added copper zone on In2.Cu, net +3.3V
- added copper zone on In1.Cu, net GND
Other:
- board outline added: 102.8 x 39.2 mm

Commit message: most of layout is done, only have single ended highspeed signals left. mika pleaaaaaaaaaaaaaaaaaseeeeeeee review :beg:
Parts:
- added JP1: Jumper_2_Small_Open, Connector_PinHeader_2.54mm:PinHeader_1x02_P2.54mm_Vertical, F.Cu at (150.5, 76.0)
- added R3: 120, Resistor_SMD:R_0603_1608Metric_Pad0.98x0.95mm_HandSolder, F.Cu at (151.8, 78.5)
- moved D1 113.1 mm to (123.8, 82.5), turned to 180 degrees
- moved R11 113.1 mm to (123.8, 84.0), turned to 180 degrees
- moved U4 108.0 mm to (125.5, 80.0), turned to 0 degrees
- moved C22 107.7 mm to (122.5, 79.2)
- moved R15 107.0 mm to (130.8, 82.2), turned to -90 degrees
- moved R17 106.5 mm to (125.5, 77.5)
- moved R14 105.1 mm to (130.8, 78.9), turned to 90 degrees
- moved J1 104.2 mm to (163.7, 71.3)
- moved J2 104.2 mm to (163.7, 94.2)
- moved C18 102.7 mm to (146.4, 87.0)
- moved Y3 102.6 mm to (153.4, 89.3), turned to 180 degrees
- moved U2 102.3 mm to (160.0, 74.8), turned to 90 degrees
- moved C20 102.1 mm to (154.2, 85.8)
- moved R16 101.6 mm to (128.5, 78.5), turned to -90 degrees
- moved C17 101.0 mm to (146.9, 82.0)
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Connections:
- J1 pad 1: /Ethernet/MDIO -> /PMOD Connector/JC1
- J1 pad 10: /PMOD Connector/JC10 -> /Ethernet/MDC
- J1 pad 2: /Ethernet/MDC -> /PMOD Connector/JC2
- J1 pad 3: /Ethernet/PHY_INT -> /PMOD Connector/JC3
- J1 pad 8: /PMOD Connector/JC8 -> /Ethernet/PHY_INT
- J1 pad 9: /PMOD Connector/JC9 -> /Ethernet/MDIO
- R10 pad 1: /PMOD Connector/JC8 -> /PMOD Connector/JC7
- R18 pad 1: /PMOD Connector/JC7 -> /PMOD Connector/JC4
- R19 pad 1: /PMOD Connector/JC4 -> /PMOD Connector/JC3
- R20 pad 1: /PMOD Connector/JC9 -> /PMOD Connector/JC2
- R21 pad 1: /PMOD Connector/JC10 -> /PMOD Connector/JC1
- R9 pad 2: /PMOD Connector/JC10 -> /PMOD Connector/JC1
- U1 pad 19: /PMOD Connector/JC8 -> /PMOD Connector/JC7
- U2 pad 1: /PMOD Connector/JC7 -> /PMOD Connector/JC4
- U2 pad 3: /PMOD Connector/JC4 -> /PMOD Connector/JC3
- U2 pad 4: /PMOD Connector/JC9 -> /PMOD Connector/JC2
- U2 pad 6: /PMOD Connector/JC10 -> /PMOD Connector/JC1
Routing:
- net GND: track 0.00 -> 52.2 mm, vias 0 -> 28
- net /Ethernet/VDDIO: track 0.00 -> 44.0 mm, vias 0 -> 4
- net VBUS: track 0.00 -> 29.5 mm, vias 0 -> 2
- net /Ethernet/RD-: track 0.00 -> 24.1 mm
- net /Ethernet/RD+: track 0.00 -> 24.1 mm
- net /Ethernet/TD-: track 0.00 -> 23.2 mm
- net /Ethernet/TD+: track 0.00 -> 23.2 mm
- net /Ethernet/LED1: track 0.00 -> 22.3 mm
- net /Ethernet/LED0: track 0.00 -> 21.4 mm, vias 0 -> 2
- net +3.3V: track 0.00 -> 19.6 mm, vias 0 -> 9
- net /Ethernet/shield: track 0.00 -> 19.3 mm
- net /PMOD Connector/JC7: track 0.00 -> 17.8 mm, vias 0 -> 2
- net Net-(J7-CC1): track 0.00 -> 14.2 mm
- net /PMOD Connector/JC4: track 0.00 -> 13.5 mm
- net Net-(J7-CC2): track 0.00 -> 13.5 mm
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- added copper zone on F.Cu, net GND
Other:
- board size 102.8 x 39.2 mm -> 80.2 x 39.2 mm
- board text added: "Differential traces must be 100Ω differential"
- board text added: "ETH_TXD[0] → JC1 ETH_TXD[1] → JC2 ETH_TX_EN → JC3 RMII_REF_CLK→ JC4 ETH_RXD[0] ← JC7 ETH_RXD[1] ← JC8 ETH_CRS_DV ← JC9"
- board text added: "Eth Differential: Trace Width: 0.2347 mm Spacing: 0.2540 mm"
- board text added: "RD+ RD- RMII_REF_CLK ETH_TXD ETH_TX_EN ETH_RXD ETH_CRS_DV"
- board text added: "Which signals are highspeed:"
- board text added: "all signal traces must be 50Ω single-ended impedance"

Commit message: finished layout + routing. needs review. still need to add testpoints
Parts:
- moved R7 0.53 mm to (139.4, 93.8)
Routing:
- net /Ethernet/MDC: track 0.00 -> 64.4 mm, vias 0 -> 1
- net /Ethernet/PHY_INT: track 2.31 -> 55.6 mm, vias 0 -> 1
- net /Ethernet/MDIO: track 1.62 -> 53.5 mm, vias 0 -> 1
- net /Ethernet/ETH_TXD1: track 0.00 -> 46.8 mm
- net /Ethernet/ETH_RXDO: track 0.00 -> 38.3 mm
- net /Ethernet/PHY_RST_N: track 1.99 -> 36.6 mm, vias 0 -> 1
- net /Ethernet/RMII_REF_CLK: track 5.68 -> 40.1 mm
- net /Ethernet/ETH_RXD1: track 0.00 -> 34.1 mm
- net /Ethernet/ETH_TXD0: track 0.00 -> 31.3 mm
- net /Ethernet/ETH_TX_EN: track 0.00 -> 28.5 mm
- net /Ethernet/ETH_CRS_DV: track 4.43 -> 31.5 mm, vias 0 -> 2
- net GND: track 52.2 -> 61.8 mm, vias 28 -> 80
- net /Ethernet/VDDIO: track 44.0 -> 38.1 mm
- added copper zone on In2.Cu, net GND
Other:
- board text added: "Single Coplanar Calcs: Track width: 0.302 mm Clearance: 0.2032 mm"
